File: tfm.kicad_pcb (KiCad board)
At the start: 2 copper layers, 100 x 90 mm, 99 parts, among them J1 Screw_Terminal_01x04, J2 Screw_Terminal_01x04, J3 Conn_01x03, J4 Conn_01x03, J5 Conn_01x03, J6 Conn_02x04_Counter_Clockwise, J7 Conn_01x02_Female, U1 LPS25HB, U10 MCP6004, U11 MCP6004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

Commit message: Add vias for ground planes
Routing:
- net GND: vias 16 -> 35
Changed lines of the file:
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@@
     (property "Sheetname" "")
     (attr exclude_from_pos_files)
-    (fp_text reference "TP2" (at 2.252 -0.048) (layer "F.SilkS")
+    (fp_text reference "TP2" (at 1.778 1.016) (layer "F.SilkS")
       (effects (font (size 0.64 0.64) (thickness 0.15)))
     )
@@
     (property "Sheetname" "")
     (attr exclude_from_pos_files)
-    (fp_text reference "TP1" (at -2.032 -0.048) (layer "F.SilkS")
+    (fp_text reference "TP1" (at -1.778 1.016) (layer "F.SilkS")
       (effects (font (size 0.64 0.64) (thickness 0.15)))
     )
@@
   (gr_line (start 98.708 102.362) (end 123.346 102.362) (layer "B.SilkS") (width 0.3))
   (gr_line (start 123.346 78.232) (end 142.65 78.232) (layer "B.SilkS") (width 0.3))
+  (gr_line (start 150.622 128.778) (end 149.606 128.778) (layer "F.SilkS") (width 0.15))
   (gr_line (start 160.176 95.758) (end 161.446 95.758) (layer "F.SilkS") (width 0.3))
+  (gr_line (start 149.606 129.794) (end 150.622 129.794) (layer "F.SilkS") (width 0.15))
   (gr_line (start 165.002 129.794) (end 165.002 131.826) (layer "F.SilkS") (width 0.15))
+  (gr_line (start 149.606 128.778) (end 149.606 126.746) (layer "F.SilkS") (width 0.15))
   (gr_line (start 165.002 131.826) (end 163.986 131.826) (layer "F.SilkS") (width 0.15))
+  (gr_line (start 150.622 131.826) (end 149.606 131.826) (layer "F.SilkS") (width 0.15))
   (gr_line (start 163.986 126.746) (end 165.002 126.746) (layer "F.SilkS") (width 0.15))
   (gr_line (start 123.346 78.232) (end 142.65 78.232) (layer "F.SilkS") (width 0.3))
   (gr_line (start 163.986 129.794) (end 165.002 129.794) (layer "F.SilkS") (width 0.15))
+  (gr_line (start 149.606 131.826) (end 149.606 129.794) (layer "F.SilkS") (width 0.15))
   (gr_line (start 178.845 95.758) (end 180.115 95.758) (layer "F.SilkS") (width 0.3))
   (gr_line (start 98.708 102.362) (end 106.328 102.362) (layer "F.SilkS") (width 0.3))
   (gr_line (start 123.346 102.362) (end 123.346 78.232) (layer "F.SilkS") (width 0.3))
+  (gr_line (start 149.606 126.746) (end 150.622 126.746) (layer "F.SilkS") (width 0.15))
   (gr_line (start 142.65 78.232) (end 142.65 95.758) (layer "F.SilkS") (width 0.3))
   (gr_line (start 165.002 126.746) (end 165.002 128.778) (layer "F.SilkS") (width 0.15))
@@
     (effects (font (size 1 1) (thickness 0.15)))
   )
+  (gr_text "C" (at 148.336 130.81) (layer "F.SilkS")
+    (effects (font (size 1 1) (thickness 0.15)))
+  )
   (gr_text "Guillermo González" (at 152.81 120.142) (layer "F.SilkS")
     (effects (font (size 2 2) (thickness 0.2)))
+  )
+  (gr_text "M" (at 148.336 127.762) (layer "F.SilkS")
+    (effects (font (size 1 1) (thickness 0.15)))
   )
   (gr_text "L1" (at 167.86 122.936) (layer "F.SilkS")
@@
   (segment (start 114.83804 64.13396) (end 114.83804 65.15204) (width 0.5) (layer "F.Cu") (net 2))
   (segment (start 124.334 61.58) (end 124.334 63.02) (width 0.5) (layer "F.Cu") (net 2))
+  (via (at 191.77 118.364) (size 0.8) (drill 0.4) (layers "F.Cu" "B.Cu") (free) (net 2))
   (via (at 124.87 83.312) (size 0.8) (drill 0.4) (layers "F.Cu" "B.Cu") (free) (net 2))
+  (via (at 140.716 125.984) (size 0.8) (drill 0.4) (layers "F.Cu" "B.Cu") (free) (net 2))
   (via (at 138.176 128.524) (size 0.8) (drill 0.4) (layers "F.Cu" "B.Cu") (free) (net 2))
   (via (at 112.424 135.636) (size 0.8) (drill 0.4) (layers "F.Cu" "B.Cu") (free) (net 2))
   (via (at 141.634 82.55) (size 0.8) (drill 0.4) (layers "F.Cu" "B.Cu") (free) (net 2))
+  (via (at 130.302 111.506) (size 0.8) (drill 0.4) (layers "F.Cu" "B.Cu") (free) (net 2))
+  (via (at 154.94 126.746) (size 0.8) (drill 0.4) (layers "F.Cu" "B.Cu") (free) (net 2))
   (via (at 124.108 80.518) (size 0.8) (drill 0.4) (layers "F.Cu" "B.Cu") (free) (net 2))
+  (via (at 114.046 124.968) (size 0.8) (drill 0.4) (layers "F.Cu" "B.Cu") (free) (net 2))
   (via (at 129.95 80.264) (size 0.8) (drill 0.4) (layers "F.Cu" "B.Cu") (net 2))
+  (via (at 128.524 113.284) (size 0.8) (drill 0.4) (layers "F.Cu" "B.Cu") (free) (net 2))
   (via (at 104.296 135.636) (size 0.8) (drill 0.4) (layers "F.Cu" "B.Cu") (free) (net 2))
+  (via (at 159.766 124.968) (size 0.8) (drill 0.4) (layers "F.Cu" "B.Cu") (free) (net 2))
+  (via (at 170.688 106.426) (size 0.8) (drill 0.4) (layers "F.Cu" "B.Cu") (free) (net 2))
+  (via (at 181.61 119.634) (size 0.8) (drill 0.4) (layers "F.Cu" "B.Cu") (free) (net 2))
+  (via (at 178.435 105.664) (size 0.8) (drill 0.4) (layers "F.Cu" "B.Cu") (free) (net 2))
+  (via (at 181.102 112.268) (size 0.8) (drill 0.4) (layers "F.Cu" "B.Cu") (free) (net 2))
+  (via (at 141.986 125.984) (size 0.8) (drill 0.4) (layers "F.Cu" "B.Cu") (free) (net 2))
   (via (at 108.868 135.636) (size 0.8) (drill 0.4) (layers "F.Cu" "B.Cu") (free) (net 2))
   (via (at 141.634 80.518) (size 0.8) (drill 0.4) (layers "F.Cu" "B.Cu") (net 2))
+  (via (at 153.416 121.92) (size 0.8) (drill 0.4) (layers "F.Cu" "B.Cu") (free) (net 2))
   (via (at 104.296 134.112) (size 0.8) (drill 0.4) (layers "F.Cu" "B.Cu") (free) (net 2))
   (via (at 140.208 130.302) (size 0.8) (drill 0.4) (layers "F.Cu" "B.Cu") (free) (net 2))
+  (via (at 132.334 111.506) (size 0.8) (drill 0.4) (layers "F.Cu" "B.Cu") (free) (net 2))
+  (via (at 191.77 120.142) (size 0.8) (drill 0.4) (layers "F.Cu" "B.Cu") (free) (net 2))
   (via (at 122.838 129.54) (size 0.8) (drill 0.4) (layers "F.Cu" "B.Cu") (free) (net 2))
   (via (at 141.634 84.582) (size 0.8) (drill 0.4) (layers "F.Cu" "B.Cu") (free) (net 2))
+  (via (at 179.832 105.664) (size 0.8) (drill 0.4) (layers "F.Cu" "B.Cu") (free) (net 2))
+  (via (at 180.086 119.634) (size 0.8) (drill 0.4) (layers "F.Cu" "B.Cu") (free) (net 2))
   (via (at 134.014 84.582) (size 0.8) (drill 0.4) (layers "F.Cu" "B.Cu") (free) (net 2))
   (via (at 110.646 135.636) (size 0.8) (drill 0.4) (layers "F.Cu" "B.Cu") (free) (net 2))
+  (via (at 155.194 121.92) (size 0.8) (drill 0.4) (layers "F.Cu" "B.Cu") (free) (net 2))
   (via (at 141.634 86.36) (size 0.8) (drill 0.4) (layers "F.Cu" "B.Cu") (free) (net 2))
+  (via (at 177.038 105.664) (size 0.8) (drill 0.4) (layers "F.Cu" "B.Cu") (free) (net 2))
   (segment (start 155.35 59.69) (end 174.654 59.69) (width 0.5) (layer "F.Cu") (net 3))
   (segment (start 170.013506 109.728) (end 174.146 109.728) (width 0.5) (layer "F.Cu") (net 3))
